Commit message: new README

File: src/gazebo_train_description/gazebo_train_description/urdf/gazebo_train.urdf (robot description, URDF)
Before this commit: robot gazebo_train, 10 links, 9 joints
Joints:
- joint camera_lens_joint: origin xyz= 0.25 0.02 0.09 rpy=-1.571 0 -1.571 -> xyz= 0.25 0.02 0.09 rpy=0 0 0

File: src/gazebo_train_description/urdf/camera.urdf.xacro (robot description, xacro)
@@ -5,5 +5,5 @@
       <origin xyz="0 0 0" rpy="${M_PI*0.5} 0 ${M_PI*0.5}"/>
       <geometry>
-        <mesh filename="package://tb3_description/meshes/webcam.stl" scale="0.0001 0.0001 0.0001"/>
+        <mesh filename="package://gazebo_train_description/meshes/webcam.stl" scale="0.0001 0.0001 0.0001"/>
       </geometry>
       <material name="red"/>

File: src/gazebo_train_description/urdf/caster.urdf.xacro (robot description, xacro)
@@ -1,5 +1,5 @@
 <?xml version="1.0"?>
-<robot xmlns:xacro="http://ros.org/wiki/xacro" name="turtlebot3_caster">
-    <xacro:macro name="turtlebot3_caster" params="alignment *origin">
+<robot xmlns:xacro="http://ros.org/wiki/xacro" name="gazebo_train_caster">
+    <xacro:macro name="gazebo_train_caster" params="alignment *origin">
         <link name="caster_back_${alignment}_link">
             <inertial>

File: src/gazebo_train_description/urdf/gazebo_train.urdf (robot description, URDF)
Before this commit: robot gazebo_train, 6 links, 5 joints
Links:
- added link camera_lens_link
- added link camera_link, mass 0.001; visual mesh filename=package://gazebo_train_description/meshes/webcam.stl scale=0.0006 0.0006 0.0006
Joints:
- added joint camera_base_joint: type fixed, parent base_link, child camera_link, origin xyz=0 0 -0.055 rpy=0 0 0
- added joint camera_lens_joint: type fixed, parent camera_link, child camera_lens_link, origin xyz=0 -0.65 0.57 rpy=-1.57 0 0 

File: src/gazebo_train_description/urdf/laser.urdf.xacro (robot description, xacro)
@@ -5,5 +5,5 @@
       <origin xyz="-0.035 0.036 0.020" rpy="${M_PI*0.5} 0 0"/>
       <geometry>
-        <mesh filename="package://tb3_description/meshes/RPLIDAR.stl" scale="0.001 0.001 0.001"/>
+        <mesh filename="package://gazebo_train_description/meshes/RPLIDAR.stl" scale="0.001 0.001 0.001"/>
       </geometry>
       <material name="red"/>

File: src/gazebo_train_description/urdf/wheel.urdf.xacro (robot description, xacro)
@@ -1,5 +1,5 @@
 <?xml version="1.0"?>
-<robot xmlns:xacro="http://ros.org/wiki/xacro" name="turtlebot3_wheel">
-    <xacro:macro name="turtlebot3_wheel" params="alignment *origin">
+<robot xmlns:xacro="http://ros.org/wiki/xacro" name="gazebo_train_wheel">
+    <xacro:macro name="gazebo_train_wheel" params="alignment *origin">
         <link name="wheel_${alignment}_link">
             <visual>
