Commit message: update train

File: src/gazebo_train_description/urdf/camera.urdf.xacro (robot description, xacro)
@@ -3,26 +3,26 @@
   <link name="camera_link">
     <visual>
-      <origin xyz="0 0 0" rpy="${M_PI*0.5} 0 ${M_PI*0.5}"/>
+        <origin xyz="0 0 0" rpy="0 0 0"/>
       <geometry>
-        <mesh filename="package://gazebo_train_description/meshes/webcam.stl" scale="0.0001 0.0001 0.0001"/>
+        <mesh filename="package://gazebo_train_description/meshes/webcam.stl" scale="0.0006 0.0006 0.0006"/>
       </geometry>
-      <material name="red"/>
+      <material name="black"/>
     </visual>
     <inertial>
       <origin xyz="0 0 0" />
-      <mass value="0.001" />
-      <inertia ixx="0.001" ixy="0.0" ixz="0.0" iyy="0.001" iyz="0.0" izz="0.001" />
+      <mass value="0.01" />
+      <inertia ixx="0.01" ixy="0.0" ixz="0.0" iyy="0.001" iyz="0.0" izz="0.001" />
     </inertial>
   </link>
-  <joint name="camera_base_joint" type="fixed">
-    <parent link="base_link"/>
-    <child link="camera_link"/>
-    <origin xyz="-0.15 -0.02 0.785" rpy="0 0 1.5"/>
-  </joint>
-  <link name="camera_lens_link"/>
-  <joint name="camera_lens_joint" type="fixed">
-    <parent link="camera_link"/>
-    <child link="camera_lens_link"/>
-    <origin xyz=" 0.25 0.02 0.09" rpy="-1.571 0 -1.571"/>
-  </joint>
+    <joint name="camera_base_joint" type="fixed">
+      <parent link="base_link"/>
+      <child link="camera_link"/>
+      <origin xyz="0 0.6 0.6" rpy="0 0 0"/>
+    </joint>
+    <link name="camera_lens_link"/>
+    <joint name="camera_lens_joint" type="fixed">
+      <parent link="camera_link"/>
+      <child link="camera_lens_link"/>
+      <origin xyz="0 0 0" rpy="-1.57 0 0 "/>
+    </joint>
 </robot>

File: src/gazebo_train_description/urdf/gazebo_train.urdf (robot description, URDF)
Before this commit: robot gazebo_train, 8 links, 7 joints
Links:
- added link imu_link
- added link laser_link
- link base_link: geometry collision mesh filename=package://gazebo_train_description/meshes/waffle_custom_bas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 scale=0.001 0.001 0.001; visual mesh filename=package://gazebo_train_description/meshes/waffle_custom_bas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 scale=0.001 0.001 0.001
Joints:
- added joint imu_joint: type fixed, parent base_link, child imu_link, origin xyz=0 0 0 rpy=0 0 0
- added joint lidar_joint: type fixed, parent base_link, child laser_link, origin xyz=0 0 0.74 rpy=0 0 3.14159, axis 0 0 1
- joint base_joint: origin xyz=0 0 0.05 rpy=0 0 0 -> xyz=0 0 0.3 rpy=0 0 0
- joint camera_base_joint: origin xyz=0 0 -0.055 rpy=0 0 0 -> xyz=0 0.6 0.6 rpy=0 0 0
- joint camera_lens_joint: origin xyz=0 -0.65 0.57 rpy=-1.57 0 0  -> xyz=0 0 0 rpy=-1.57 0 0 
- joint wheel_left2_joint: origin xyz=-0.22 0.400 0.05 rpy=-1.5707963267948966 0 0  -> xyz=-0.22 0.400 0.1 rpy=-1.5707963267948966 0 0 
- joint wheel_left_joint: origin xyz=-0.220  -0.400 0.05 rpy=-1.5707963267948966 0 0 -> xyz=-0.220  -0.400 0.1 rpy=-1.5707963267948966 0 0
- joint wheel_right2_joint: origin xyz=0.22 0.400 0.05 rpy=-1.5707963267948966 0 -3.141592653589793  -> xyz=0.22 0.400 0.1 rpy=-1.5707963267948966 0 -3.141592653589793 
- joint wheel_right_joint: origin xyz=0.22 -0.400 0.05 rpy=-1.5707963267948966 0 -3.141592653589793 -> xyz=0.22 -0.400 0.1 rpy=-1.5707963267948966 0 -3.141592653589793

File: src/gazebo_train_description/urdf/gazebo_train.urdf.xacro (robot description, xacro)
@@ -3,5 +3,5 @@
 	<!-- common constants -->
   <xacro:include filename="$(find gazebo_train_description)/urdf/common_properties.xacro"/>
-	<!-- Turtlebot3 platform include files -->
+	<!-- gazebo_train platform include files -->
   <xacro:include filename="$(find gazebo_train_description)/urdf/wheel.urdf.xacro"/>
 	<!-- Base -->
@@ -10,41 +10,41 @@
     <parent link="base_footprint"/>
     <child link="base_link" />
-    <origin xyz="0 0 -0.030" rpy="0 0 0"/>
+    <origin xyz="0 0 0.30" rpy="0 0 0"/>
   </joint>
   <link name="base_link">
     <visual>
-      <origin xyz="-0.235 -0.278 0.285" rpy="0 0.01 0"/>
+      <origin xyz="0 0 0.25" rpy="0 0 0"/>
       <geometry>
-        <mesh filename="package://gazebo_train_description/meshes/waffle_custom_base.stl" scale="0.001 0.001 0.001"/>		<!-- make sure that the path points correctly to the mesh file -->
+        <mesh filename="package://gazebo_train_description/meshes/waffle_custom_base.stl" scale="0.001 0.001 0.001"/>
       </geometry>
       <material name="dark"/>
     </visual>
     <collision>
-      <origin xyz="-0.10 0 0.07" rpy="0 0.01 0"/>
+      <origin xyz="0 0 0.25" rpy="0 0 0"/>
       <geometry>
-        <box size="0.27 0.11 0.27"/>
+        <mesh filename="package://gazebo_train_description/meshes/waffle_custom_base.stl" scale="0.001 0.001 0.001"/>
       </geometry>
     </collision>
     <inertial>
-      <origin xyz="-0.10 0 0.07" rpy="0 0.01 0"/>
-      <mass value="1"/>
-      <inertia ixx="0.0270833333" ixy="0.0" ixz="0.0"
-               iyy="0.01215" iyz="0.0"
-               izz="0.0270833333" />
+      <origin xyz="0 0 0.3" rpy="0 0 0"/>
+      <mass value="3"/>
+      <inertia ixx="0.6" ixy="0.0" ixz="0.0"
+               iyy="0.2" iyz="0.0"
+               izz="0.6" />
     </inertial>
   </link>
-	<!-- Turtlebot3 wheel macros -->
-<xacro:turtlebot3_wheel alignment="left">
-  <origin xyz="-0.455  -0.678 0.1350" rpy="${-M_PI*0.5} 0 0"/>
-</xacro:turtlebot3_wheel>
-<xacro:turtlebot3_wheel alignment="right">
-  <origin xyz="-0.455  0.123 0.1350" rpy="${-M_PI*0.5} 0 0"/>
-</xacro:turtlebot3_wheel>
-<xacro:turtlebot3_wheel alignment="right2">
-  <origin xyz="-0.015 0.123 0.1350" rpy="${-M_PI*0.5} 0 ${-M_PI} "/>
-</xacro:turtlebot3_wheel>
-<xacro:turtlebot3_wheel alignment="left2">
-  <origin xyz="-0.015 -0.678 0.1350" rpy="${-M_PI*0.5} 0 ${-M_PI} "/>
-</xacro:turtlebot3_wheel>
+	<!-- gazebo_train wheel macros -->
+<xacro:gazebo_train_wheel alignment="left">
+  <origin rpy="-1.5707963267948966 0 0" xyz="-0.220  -0.400 0.1"/>
+</xacro:gazebo_train_wheel>
+<xacro:gazebo_train_wheel alignment="right">
+  <origin rpy="-1.5707963267948966 0 -3.141592653589793" xyz="0.22 -0.400 0.1"/>
+</xacro:gazebo_train_wheel>
+<xacro:gazebo_train_wheel alignment="right2">
+  <origin rpy="-1.5707963267948966 0 -3.141592653589793 " xyz="0.22 0.400 0.1"/>
+</xacro:gazebo_train_wheel>
+<xacro:gazebo_train_wheel alignment="left2">
+  <origin rpy="-1.5707963267948966 0 0 " xyz="-0.22 0.400 0.1"/>
+</xacro:gazebo_train_wheel>
 	<!-- sensors -->
 <xacro:include filename="$(find gazebo_train_description)/urdf/camera.urdf.xacro"/>

File: src/gazebo_train_description/urdf/imu.urdf.xacro (robot description, xacro)
@@ -5,5 +5,5 @@
     <parent link="base_link"/>
     <child link="imu_link"/>
-    <origin xyz="-0.25 -0.250 0.468" rpy="0 0 0"/>
+    <origin xyz="0 0 0" rpy="0 0 0"/>
   </joint>
 </robot>

File: src/gazebo_train_description/urdf/laser.urdf.xacro (robot description, xacro)
@@ -1,28 +1,43 @@
 <?xml version="1.0"?>
 <robot>
-  <link name="laser_link">
-    <visual>
-      <origin xyz="-0.035 0.036 0.020" rpy="${M_PI*0.5} 0 0"/>
-      <geometry>
-        <mesh filename="package://gazebo_train_description/meshes/RPLIDAR.stl" scale="0.001 0.001 0.001"/>
-      </geometry>
-      <material name="red"/>
-    </visual>
-    <inertial>
-      <origin xyz="0 0 0" />
-      <mass value="0.2" />
-      <inertia ixx="0.001" ixy="0.0" ixz="0.0" iyy="0.001" iyz="0.0" izz="0.001" />
-    </inertial>
-    <collision>
-      <origin xyz="0 0 0" rpy="${M_PI*0.5} 0 0"/>
-      <geometry>
-        <box size="0.1 0.056 0.420"/>
-      </geometry>
-    </collision>
-  </link>
-  <joint name="laser_joint" type="fixed">
-    <parent link="base_link"/>
-    <child link="laser_link"/>
-    <origin xyz="-0.02 0 0.80" rpy="0 0 0"/>
-  </joint>
-</robot>
+    <link name="laser_link">
+      <sensor name="hls_lfcd_lds" type="ray">
+        <always_on>true</always_on>
+        <visualize>false</visualize>
+        <pose>0 0 0 0 0 0</pose>
+        <update_rate>10</update_rate>
+        <ray>
+          <scan>
+            <horizontal>
+              <samples>1024</samples>
+              <resolution>1.000000</resolution>
+              <min_angle>0.000000</min_angle>
+              <max_angle>6.280000</max_angle>
+            </horizontal>
+          </scan>
+          <range>
+            <min>0.5</min>
+            <max>120</max>
+            <resolution>0.0010000</resolution>
+          </range>
+          <noise>
+            <type>gaussian</type>
+            <mean>0.0</mean>
+            <stddev>0.01</stddev>
+          </noise>
+        </ray>
+        <plugin name="train_laserscan" filename="libgazebo_ros_ray_sensor.so">
+          <ros>
+            <remapping>~/out:=scan</remapping>
+          </ros>
+          <output_type>sensor_msgs/LaserScan</output_type>
+          <frame_name>base_footprint</frame_name>
+        </plugin>
+      </sensor>
+    </link>
+    <joint name="lidar_joint" type="fixed">
+        <parent link="base_link"/>
+        <child link="laser_link"/>
+        <origin rpy="0 0 3.14159" xyz="0 0 0.74"/>
+        <axis xyz="0 0 1"/>
+    </joint>

File: src/gazebo_train_description/urdf/wheel.urdf.xacro (robot description, xacro)
@@ -4,5 +4,5 @@
         <link name="wheel_${alignment}_link">
             <visual>
-                <origin xyz="0 0 0" rpy="${M_PI*0.5} 0 0"/>
+                <origin xyz="1.5708 0 0" rpy="${M_PI*0.5} 0 0"/>
                 <geometry>
                     <mesh filename="package://gazebo_train_description/meshes/${alignment}_tire.stl" scale="0.001 0.001 0.001"/>
@@ -16,7 +16,7 @@
             </inertial>
             <collision>
-                <origin rpy="0 0 0" xyz="0 0 0"/>
+                <origin rpy="-1.5708 0 0" xyz="0 0 0"/>
                 <geometry>
-                    <cylinder length="0.1" radius="0.1"/>
+                    <mesh filename="package://gazebo_train_description/meshes/${alignment}_tire.stl" scale="0.001 0.001 0.001"/>
                 </geometry>
             </collision>
@@ -26,5 +26,4 @@
             <child link="wheel_${alignment}_link"/>
             <xacro:insert_block name="origin"/>
-            <axis xyz="0 0 1"/>
         </joint>
     </xacro:macro>
