Commit message: update readme and clean project

File: src/gazebo_train_description/urdf/gazebo_train.urdf (robot description, URDF)
Before this commit: robot gazebo_train, 10 links, 9 joints
Links:
- link base_link: geometry collision mesh filename=package://gazebo_train_description/meshes/gazebo_train_base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 scale=0.001 0.001 0.001; visual mesh filename=package://gazebo_train_description/meshes/gazebo_train_base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 scale=0.001 0.001 0.001
